File: Hydrophone.kicad_pcb (KiCad board)
At the start: 2 copper layers, 26 x 26 mm, 36 parts, among them J201 USB_C_Receptacle_USB2.0_16P, U201 PCM2912APJTR, U202 OPA1642AIDR, X201 6MHz

Commit message: repo as manufactured
Parts:
- removed C212: 0.22u, Capacitor_SMD:CP_Elec_6.3x5.4
- added C201: 22u, Capacitor_SMD:C_0805_2012Metric, F.Cu at (148.0, 104.9)
- added C203: 100n, Capacitor_SMD:C_0402_1005Metric, F.Cu at (134.9, 108.4)
- added C204: 22u, Capacitor_SMD:C_0805_2012Metric, F.Cu at (139.4, 109.6)
- added C401: 3.3u, Capacitor_Tantalum_SMD:CP_EIA-3216-18_Kemet-A, F.Cu at (151.5, 65.3)
- added C402: 1u, Capacitor_SMD:C_0402_1005Metric, F.Cu at (139.7, 67.2)
- added C403: 100n, Capacitor_SMD:C_0402_1005Metric, F.Cu at (140.8, 67.2)
- added C404: 100n, Capacitor_SMD:C_0402_1005Metric, F.Cu at (141.8, 67.2)
- added C405: 1u, Capacitor_SMD:C_0402_1005Metric, F.Cu at (145.6, 49.9)
- added C406: 1u, Capacitor_SMD:C_0402_1005Metric, F.Cu at (152.5, 61.3)
- added C407: 1u, Capacitor_SMD:C_0402_1005Metric, F.Cu at (150.0, 49.3)
- added C408: 3.3u, Capacitor_Tantalum_SMD:CP_EIA-3216-18_Kemet-A, F.Cu at (151.5, 63.0)
- added C409: 100p, Capacitor_SMD:C_0402_1005Metric, F.Cu at (147.5, 61.7)
- added C410: 100p, Capacitor_SMD:C_0402_1005Metric, F.Cu at (148.6, 61.7)
- added C411: 100n, Capacitor_SMD:C_0402_1005Metric, F.Cu at (150.5, 61.3)
- added C412: 1u, Capacitor_SMD:C_0402_1005Metric, F.Cu at (141.7, 55.5)
- added C413: 30p, Capacitor_SMD:C_0402_1005Metric, F.Cu at (141.2, 57.2)
- added C414: 30p, Capacitor_SMD:C_0402_1005Metric, F.Cu at (143.4, 58.1)
- added C415: 22u, Capacitor_SMD:C_0805_2012Metric, F.Cu at (143.8, 69.5)
- added D201: 12v Zener, Diode_SMD:D_SOD-123, F.Cu at (145.3, 110.5)
- added D202: 12v Zener, Diode_SMD:D_SOD-123, F.Cu at (150.4, 110.5)
- added D301: 6.8v Zener, Diode_SMD:D_SOD-123, F.Cu at (136.8, 114.7)
- added D302: 6.8v Zener, Diode_SMD:D_SOD-123, F.Cu at (135.6, 118.6)
- added D401: 6.8v Zener, Diode_SMD:D_SOD-123, F.Cu at (147.8, 71.0)
- added D402: 6.8v Zener, Diode_SMD:D_SOD-123, F.Cu at (147.8, 66.0)
- added J201: AudioJack4, Connector_Audio:Jack_3.5mm_PJ320D_Horizontal, B.Cu at (147.2, 107.0)
- added J301: AudioJack4, Connector_Audio:Jack_3.5mm_PJ320D_Horizontal, F.Cu at (147.2, 118.0)
- added J401: USB_C_Receptacle_USB2.0_16P, Connector_USB:USB_C_Receptacle_G-Switch_GT-USB-7025, F.Cu at (132.9, 53.6)
- added L401: 1uH, Inductor_SMD:L_1210_3225Metric, F.Cu at (142.1, 51.4)
- added Q301: MMBFJ201, Package_TO_SOT_SMD:SOT-23, F.Cu at (138.9, 118.0)
- added Q401: MMBFJ201, Package_TO_SOT_SMD:SOT-23, F.Cu at (140.0, 70.4)
- added R101: 0, Resistor_SMD:R_0603_1608Metric, B.Cu at (144.9, 92.6)
- added R103: 0, Resistor_SMD:R_0603_1608Metric, B.Cu at (149.5, 95.5)
- added R201: 47, Resistor_SMD:R_0805_2012Metric, F.Cu at (151.5, 104.9)
- added R202: 1k, Capacitor_SMD:C_0402_1005Metric, F.Cu at (132.8, 104.9)
- added R203: 10k, Resistor_SMD:R_1206_3216Metric, F.Cu at (148.5, 107.5)
- added R204: 10M, Resistor_SMD:R_0402_1005Metric, F.Cu at (132.8, 106.9)
- added R205: 1k, Capacitor_SMD:C_0402_1005Metric, F.Cu at (141.7, 106.9)
- added R206: 47k, Resistor_SMD:R_0402_1005Metric, F.Cu at (137.4, 108.4)
- added R207: 47k, Resistor_SMD:R_0402_1005Metric, F.Cu at (135.9, 109.5)
- added R301: 10M, Resistor_SMD:R_0402_1005Metric, F.Cu at (138.5, 120.4)
- added R401: 1k5, Resistor_SMD:R_0402_1005Metric, F.Cu at (142.8, 67.2)
- added R402: 10M, Resistor_SMD:R_0402_1005Metric, F.Cu at (154.7, 66.9)
- added R403: 0, Resistor_SMD:R_0603_1608Metric, B.Cu at (153.6, 49.4)
- added R404: 47k, Resistor_SMD:R_0402_1005Metric, F.Cu at (145.1, 65.4)
- added R405: 0, Resistor_SMD:R_0603_1608Metric, F.Cu at (152.6, 49.4)
- added R406: 47k, Resistor_SMD:R_0402_1005Metric, F.Cu at (148.0, 49.3)
- added R407: 33, Resistor_SMD:R_0402_1005Metric, F.Cu at (144.0, 53.9)
- added R408: 33, Resistor_SMD:R_0402_1005Metric, F.Cu at (144.0, 54.9)
- added R409: 1k5, Resistor_SMD:R_0402_1005Metric, F.Cu at (144.0, 56.0)
- added R410: 1M, Resistor_SMD:R_0402_1005Metric, F.Cu at (144.5, 57.9)
- added R411: 5k1, Resistor_SMD:R_0402_1005Metric, F.Cu at (138.3, 52.2)
- added R412: 5k1, Resistor_SMD:R_0402_1005Metric, F.Cu at (138.3, 56.3)
- added REF**: Slot, Mouse_Bites:Slot, F.Cu at (143.0, 100.6)
- added REF**: Mouse Bites, Mouse_Bites:Mouse Bites, F.Cu at (135.6, 99.7)
- added REF**: Slot, Mouse_Bites:Slot, F.Cu at (131.2, 111.6)
- added REF**: Slot, Mouse_Bites:Slot, F.Cu at (154.8, 73.6)
- added REF**: Mouse Bites, Mouse_Bites:Mouse Bites, F.Cu at (150.4, 72.7)
- added REF**: Slot, Mouse_Bites:Slot, F.Cu at (131.2, 73.6)
- added REF**: Slot, Mouse_Bites:Slot, F.Cu at (143.0, 73.6)
- added REF**: Mouse Bites, Mouse_Bites:Mouse Bites, F.Cu at (135.6, 72.7)
- added REF**: Mouse Bites, Mouse_Bites:Mouse Bites, F.Cu at (150.4, 99.7)
- added REF**: Mouse Bites, Mouse_Bites:Mouse Bites, F.Cu at (150.4, 110.7)
- added REF**: Slot, Mouse_Bites:Slot, F.Cu at (154.8, 111.6)
- added REF**: Slot, Mouse_Bites:Slot, F.Cu at (131.2, 100.6)
- added REF**: Slot, Mouse_Bites:Slot, F.Cu at (154.8, 100.6)
- added REF**: Mouse Bites, Mouse_Bites:Mouse Bites, F.Cu at (135.6, 110.7)
- added REF**: Slot, Mouse_Bites:Slot, F.Cu at (143.0, 111.6)
- added TP201: PEIZO+, TestPoint:TestPoint_Pad_D1.0mm, F.Cu at (131.0, 105.4)
- added TP202: PEIZO-, TestPoint:TestPoint_Pad_D1.0mm, F.Cu at (131.0, 108.5)
- added TP203: PEIZO+, TestPoint:TestPoint_Pad_D1.0mm, F.Cu at (155.0, 103.0)
- added TP204: PEIZO-, TestPoint:TestPoint_Pad_D1.0mm, F.Cu at (155.0, 105.5)
- added TP205: PEIZO+, TestPoint:TestPoint_Pad_D1.0mm, F.Cu at (155.0, 111.0)
- added TP206: PEIZO-, TestPoint:TestPoint_Pad_D1.0mm, F.Cu at (155.0, 108.4)
- added TP301: PEIZO+, TestPoint:TestPoint_Pad_D1.0mm, F.Cu at (131.0, 116.3)
- added TP302: PEIZO-, TestPoint:TestPoint_Pad_D1.0mm, F.Cu at (131.0, 119.4)
- added TP401: PEIZO+, TestPoint:TestPoint_Pad_D1.0mm, F.Cu at (155.0, 63.5)
- added TP402: PEIZO-, TestPoint:TestPoint_Pad_D1.0mm, F.Cu at (155.0, 60.5)
- added U201: OPA1642AIDR, OPA1642AIDR:D8, F.Cu at (137.2, 105.1)
- added U401: PCM2912APJTR, PCM2912A:PJT32, F.Cu at (150.3, 55.5)
- added X401: 6MHz, Crystal:Crystal_SMD_HC49-SD, F.Cu at (139.4, 61.8)
- L101: renamed from L201; value 1u -> 1uH
- R106: renamed from R210; value 1M -> 10M
- renumbered C211 to C101, C213 to C103, C214 to C104, C201 to C105, C202 to C106, C203 to C107, C204 to C108, C205 to C109, C206 to C110, C207 to C111, C208 to C112, C209 to C113, C210 to C114, D201 to D101, D202 to D102, J201 to J101, R205 to R102, R208 to R104, R209 to R105, R211 to R107, R201 to R108, R202 to R109, R203 to R110, R204 to R111, R206 to R112, R207 to R113, R212 to R114, R213 to R115, TP201 to TP101, TP202 to TP102, U202 to U101, U201 to U102, X201 to X101
Routing:
- net VBUS_2: track 0.00 -> 28.1 mm, vias 0 -> 2
- net Net-(D201-K): track 0.00 -> 27.7 mm, vias 0 -> 2
- net /9V_To_3.5mm_Jack/Jack+: track 0.00 -> 27.3 mm, vias 0 -> 1
- net /USBC_Out_No_OPAMP/MBIAS: track 0.00 -> 25.2 mm, vias 0 -> 2
- net GNDA_4: track 0.00 -> 21.8 mm, vias 0 -> 23
- net Net-(U401A-MAMP): track 0.00 -> 21.8 mm, vias 0 -> 3
- net /USBC_Out_No_OPAMP/Peizo+: track 0.00 -> 20.8 mm
- net VGND_2: track 0.00 -> 18.0 mm, vias 0 -> 2
- net /USBC_Out_No_OPAMP/MIC_AFTER_JFET: track 0.00 -> 17.8 mm
- net Net-(D301-A): track 0.00 -> 16.1 mm
- net Net-(U401A-XTO): track 0.00 -> 13.9 mm
- net /9V_To_3.5mm_Jack/INA-: track 0.00 -> 13.3 mm, vias 0 -> 2
- net Net-(U401B-POWER): track 0.00 -> 12.7 mm, vias 0 -> 2
- net GNDA_2: track 0.00 -> 12.6 mm, vias 0 -> 12
- net VBUS_4: track 0.00 -> 12.0 mm
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- added copper zone on B.Cu, net GNDA_2
- added copper zone on F.Cu, net GNDA_2
- added copper zone on B.Cu, net GNDA_3
- added copper zone on F.Cu, net GNDA_3
- added copper zone on B.Cu, net GNDA_4
- added copper zone on F.Cu, net GNDA_4
Other:
- board size 26 x 26 mm -> 26 x 75 mm
- board text added: "+"
- board text added: "+9V"
- board text added: "-"
- board text added: "Jack"
- board text added: "PEIZO"
- board text added: "Remus Harris Peizoelectric Amp Rev1, 2/15/2025"
- board text added: "bridge"
