File: 9V_To_3.5mm_Jack.kicad_sch (KiCad schematic)
At the start: 20 parts, among them J201 AudioJack4, U201 OPA1642AIDR

Commit message: fixed BOM to correct part number for 47ohm 0805 resistor. New file sent to JLCPCB for manufacturing
Parts:
- R201: JLCPCB Part# C17902 -> C17714; Part Number 1206W4F1002T5E -> 0805W8F470JT5E
Changed lines of the file:
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@@
 			)
 		)
-		(property "Part Number" "1206W4F1002T5E"
+		(property "Part Number" "0805W8F470JT5E"
 			(at 114.3 33.02 0)
 			(effects
@@
 			)
 		)
-		(property "JLCPCB Part#" "C17902"
+		(property "JLCPCB Part#" "C17714"
 			(at 114.3 33.02 0)
 			(effects
