File: USBC_Out.kicad_sch (KiCad schematic)
At the start: 36 parts, among them J201 USB_C_Receptacle_USB2.0_16P, U201 PCM2912APJTR, U202 OPA1642AIDR, X201 6MHz

Commit message: repo as manufactured
Parts:
- removed C212: 0.22u, Capacitor_SMD:CP_Elec_6.3x5.4, symbol Device:C_Polarized
- added R101, R103: 0, Resistor_SMD:R_0603_1608Metric, symbol Device:R
- C101: renamed from C211; JLCPCB Part# (none) -> C45783
- C103: renamed from C213; JLCPCB Part# (none) -> C1525
- C104: renamed from C214; JLCPCB Part# (none) -> C45783
- C105: renamed from C201; JLCPCB Part# (none) -> C52923
- C106: renamed from C202; JLCPCB Part# (none) -> C52923
- C107: renamed from C203; JLCPCB Part# (none) -> C52923
- C108: renamed from C204; JLCPCB Part# (none) -> C7184
- C109: renamed from C205; JLCPCB Part# (none) -> C1546
- C110: renamed from C206; JLCPCB Part# (none) -> C1546
- C111: renamed from C207; JLCPCB Part# (none) -> C1525
- C112: renamed from C208; JLCPCB Part# (none) -> C52923
- C113: renamed from C209; JLCPCB Part# (none) -> C1570
- C114: renamed from C210; JLCPCB Part# (none) -> C1570
- D101: renamed from D201; JLCPCB Part# (none) -> C2120
- D102: renamed from D202; JLCPCB Part# (none) -> C2120
- J101: renamed from J201; JLCPCB Part# (none) -> C963213
- L101: renamed from L201; value 1u -> 1uH; JLCPCB Part# (none) -> C22202
- R102: renamed from R205; JLCPCB Part# (none) -> C17902
- R104: renamed from R208; JLCPCB Part# (none) -> C11702
- R105: renamed from R209; JLCPCB Part# (none) -> C17902
- R106: renamed from R210; value 1M -> 10M; JLCPCB Part# (none) -> C26082; Part Number 0402WGF1004TCE -> 0402WGF1005TCE
- R107: renamed from R211; JLCPCB Part# (none) -> C11702
- R108: renamed from R201; JLCPCB Part# (none) -> C25105
- R109: renamed from R202; JLCPCB Part# (none) -> C25105
- R110: renamed from R203; JLCPCB Part# (none) -> C25930
- R111: renamed from R204; JLCPCB Part# (none) -> C26083
- R112: renamed from R206; JLCPCB Part# (none) -> C25905
- R113: renamed from R207; JLCPCB Part# (none) -> C25905
- R114: renamed from R212; JLCPCB Part# (none) -> C25792
- R115: renamed from R213; JLCPCB Part# (none) -> C25792
- TP101: renamed from TP201; Part Number (none) -> ---
- TP102: renamed from TP202; Part Number (none) -> ---
- U101: renamed from U202; JLCPCB Part# (none) -> C67640; Part Number (none) -> OPA1642AIDR
- U102: renamed from U201; JLCPCB Part# (none) -> C475497; Part Number (none) -> PCM2912APJTR
- X101: renamed from X201; JLCPCB Part# (none) -> C7528811
Connections:
- net OPAMP_MIC: now also R101.2, R103.2
- net at R102.2: now also R103.1
- net at C101.1, R102.1: now also R101.1
Other:
- note added: "Solderbridge when bringing up board"
- moved on the sheet: C113, C114, R108, R109, R111, U102A, X101

Commit message: fixed BOM to correct part number for 47ohm 0805 resistor. New file sent to JLCPCB for manufacturing
Parts:
- R102: JLCPCB Part# C17902 -> C17714; Part Number 1206W4F1002T5E -> 0805W8F470JT5E
Changed lines of the file:
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@@
 			)
 		)
-		(property "Part Number" "1206W4F1002T5E"
+		(property "Part Number" "0805W8F470JT5E"
 			(at 118.11 123.19 0)
 			(effects
@@
 			)
 		)
-		(property "JLCPCB Part#" "C17902"
+		(property "JLCPCB Part#" "C17714"
 			(at 118.11 123.19 0)
 			(effects
